File: Schematics/SMuFF Relay board/Relay-Board.kicad_pcb (KiCad board)
At the start: 2 copper layers, 56.9 x 22 mm, 13 parts, among them J1 JST XH, J2 JST XH, J3 JST XH, J4 JST XH, K1 G6A-274P, K2 G6A-274P, Q1 BC847/547, Q2 BC847/547, U1 TLP521

Commit message: Updated Relay-Board PCB
Routing:
- net Net-(J3-Pad4): track 39.0 -> 42.6 mm
- net Net-(J3-Pad3): track 42.3 -> 41.3 mm
- net Net-(J2-Pad2): track 10.1 -> 9.45 mm
- added copper zone on B.Cu, net Net-(J1-Pad4)
Other:
- net class Relay added: clearance 0.5, trace_width 0.5, via_dia 1, via_drill 0.4

Commit message: Updated to V3.12; See README.md
Other:
- net class Default removed
- net class Relay removed
- rule pad_to_mask_clearance: 0.051 -> 0

Commit message: Updated for arduino framework 2.4.0
Parts:
- D1, D2: footprint Diode_SMD:D_0603_1608Metric -> Diode_SMD:D_SOD-123
Routing:
- net Net-(D1-Pad1): track 58.2 -> 56.5 mm
- net Net-(D2-Pad2): track 42.4 -> 41.5 mm
- net Net-(D1-Pad2): track 12.9 -> 12.4 mm
Other:
- board text added: "2020-2023 by Technik Gegg"
- board text added: "Rev:2"
- board text removed: "2020 by Technik Gegg"
- board text removed: "Rev:1"
